File: anice.kicad_pcb (KiCad board)
At the start: 4 copper layers, 65 x 34 mm, 92 parts, among them J1 Conn_02x20_Counter_Clockwise, J2 Micro_SD_Card_Det1, J3 USB_C_Receptacle_USB2.0_14P, J4 USB_C_Receptacle_USB2.0_14P, J5 USB_C_Receptacle_USB2.0_14P, J7 HDMI_C_1.3, U1 ECP5U_12_CABGA256, U10 W9825G6KH-6, U11 W25Q128JVS, U12 TLV62569DRL, U13 TLV62569DRL, U14 TLV62569DRL, U5 TPD2EUSB30, U6 TPD2EUSB30, U7 FT231XQ, U8 TPD2EUSB30, U9 PCA9306DC1, Y1 ECS-2520MV-xxx-xx

Commit message: Rev 1
Parts:
- added C22: 22uF, Capacitor_SMD:C_0603_1608Metric, B.Cu at (106.7, 83.5)
- added R38: 0.47, Resistor_SMD:R_0603_1608Metric, B.Cu at (106.7, 82.0)
- moved C25 1.29 mm to (134.6, 84.3), turned to -90 degrees
- moved C26 0.74 mm to (133.3, 86.5)
Connections:
- J2 pad 1: unconnected-(J2-DAT2-Pad1) -> SD_D2
- J2 pad 10: unconnected-(J2-DET_A-Pad10) -> SD_DET
- J2 pad 11: unconnected-(J2-SHIELD-Pad11) -> GND
- J2 pad 2: unconnected-(J2-DAT3/CD-Pad2) -> SD_D3
- J2 pad 3: unconnected-(J2-CMD-Pad3) -> SD_CMD
- J2 pad 4: unconnected-(J2-VDD-Pad4) -> Net-(J2-VDD)
- J2 pad 5: unconnected-(J2-CLK-Pad5) -> SD_CLK
- J2 pad 6: unconnected-(J2-VSS-Pad6) -> GND
- J2 pad 7: unconnected-(J2-DAT0-Pad7) -> SD_D0
- J2 pad 8: unconnected-(J2-DAT1-Pad8) -> SD_D1
- J2 pad 9: unconnected-(J2-DET_B-Pad9) -> GND
- U1 pad E4: unconnected-(U1B-PT9A/+-PadE4) -> CONN33
- U1 pad F15: D2+ -> unconnected-(U1D-PR11C/+/RDQ8-PadF15)
- U1 pad F16: D2- -> D2+
- U1 pad F2: unconnected-(U1G-PL11C/+/LDQ8-PadF2) -> CONN38
- U1 pad F3: unconnected-(U1G-PL5D/-/LDQ8-PadF3) -> CONN27
- U1 pad F4: unconnected-(U1G-PL8C/+/LDQ8-PadF4) -> CONN29
- U1 pad G1: unconnected-(U1G-PL20A/+/GR_PCLK7_1/HS/LDQS20-PadG1) -> CONN36
- U1 pad G15: D3+ -> D2-
- U1 pad G2: unconnected-(U1G-PL14B/-/HS/LDQ20-PadG2) -> CONN31
- U1 pad H15: unconnected-(U1D-PR20B/-/HS/RDQSN20-PadH15) -> D3+
- U1 pad J1: unconnected-(U1G-PL23A/+/PCLKT7_1/HS/LDQ20-PadJ1) -> CONN32
- U1 pad J2: unconnected-(U1G-PL23B/-/PCLKC7_1/HS/LDQ20-PadJ2) -> CONN23
- U1 pad K1: unconnected-(U1G-PL23C/+/PCLKT7_0/LDQ20-PadK1) -> CONN28
- U1 pad K2: unconnected-(U1G-PL23D/-/PCLKC7_0/LDQ20-PadK2) -> CONN26
- U1 pad L1: unconnected-(U1F-PL26A/+/PCLKT6_1/HS/LDQ32-PadL1) -> CONN21
- U1 pad L2: unconnected-(U1F-PL26B/-/PCLKC6_1/HS/LDQ32-PadL2) -> CONN24
- U1 pad L3: unconnected-(U1F-PL32C/+/LDQ32-PadL3) -> CONN13
- U1 pad L4: unconnected-(U1F-PL29C/+/GR_PCLK6_1/LDQ32-PadL4) -> SD_CLK
- U1 pad M1: unconnected-(U1F-PL26C/+/PCLKT6_0/LDQ32-PadM1) -> CONN22
- U1 pad M2: unconnected-(U1F-PL26D/-/PCLKC6_0/LDQ32-PadM2) -> CONN19
- U1 pad M3: unconnected-(U1F-PL32D/-/LDQ32-PadM3) -> CONN11
- U1 pad N1: unconnected-(U1F-PL32A/+/HS/LDQS32-PadN1) -> CONN18
- U1 pad N4: unconnected-(U1F-PL38A/+/HS/LDQ44-PadN4) -> SD_D2
- U1 pad P1: unconnected-(U1F-PL35A/+/HS/LDQ32-PadP1) -> CONN12
- U1 pad P16: FPDI_CEC -> FPDI_D0+
- U1 pad P2: unconnected-(U1F-PL32B/-/HS/LDQSN32-PadP2) -> CONN10
- U1 pad P3: unconnected-(U1F-PL38B/-/HS/LDQ44-PadP3) -> CONN16
- U1 pad P4: unconnected-(U1F-PL41A/+/HS/LDQ44-PadP4) -> SD_D3
- U1 pad R12: unconnected-(U1E-PR44A/+/HS/RDQS44-PadR12) -> FPDI_CEC
- U1 pad R15: FPDI_D0- -> FPDI_CLK-
- U1 pad R16: FPDI_D0+ -> FPDI_D0-
- U1 pad T14: FPDI_CLK- -> unconnected-(U1E-PR41D/-/RDQ44-PadT14)
- U1 pad T4: unconnected-(U1F-PL44B/-/HS/LDQSN44-PadT4) -> SD_D0
- U1 pad T6: unconnected-(U1H-PB4A/+/D7/IO7-PadT6) -> SD_D1
Routing:
- net SD_D2: track 0.00 -> 32.9 mm, vias 0 -> 2
- net SD_CLK: track 0.00 -> 32.3 mm, vias 0 -> 2
- net SD_D3: track 0.00 -> 31.3 mm, vias 0 -> 2
- net SD_D1: track 0.00 -> 29.6 mm, vias 0 -> 2
- net SD_CMD: track 0.00 -> 28.9 mm, vias 0 -> 2
- net SD_D0: track 0.00 -> 28.2 mm, vias 0 -> 2
- net +2V5: track 53.1 -> 25.3 mm, vias 6 -> 5
- net CONN38: track 0.00 -> 25.1 mm
- net CONN36: track 0.00 -> 22.0 mm
- net CONN32: track 0.00 -> 18.8 mm
- net CONN10: track 0.00 -> 18.2 mm
- net CONN33: track 0.00 -> 18.0 mm, vias 0 -> 1
- net CONN31: track 0.00 -> 16.5 mm
- net CONN11: track 0.00 -> 15.5 mm, vias 0 -> 1
- net CONN28: track 0.00 -> 15.2 mm
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
Commit message: No DRC Errors
Parts:
- moved H2 0.60 mm to (164.1, 74.5)
- moved H4 0.60 mm to (164.1, 101.5)
- moved U6 0.06 mm to (137.4, 97.1)
Connections:
- J2 pad 10: SD_DET -> unconnected-(J2-DET_A-Pad10)
- U1 pad R12: FPDI_CEC -> unconnected-(U1E-PR44A/+/HS/RDQS44-PadR12)
- U1 pad R5: unconnected-(U1F-PL44A/+/HS/LDQS44-PadR5) -> SD_CMD
- U1 pad T14: unconnected-(U1E-PR41D/-/RDQ44-PadT14) -> FPDI_CEC
Routing:
- net GND: track 85.9 -> 94.4 mm, vias 59 -> 60
- net +1V1: track 45.2 -> 52.6 mm
- net FT2V5: track 14.6 -> 21.2 mm, vias 0 -> 2
- net D2+: track 21.6 -> 17.7 mm
- net SD_CMD: track 28.9 -> 31.1 mm
- net SD_DET: track 2.15 -> 0.00 mm, vias 1 -> 0
- net +3V3: track 74.5 -> 76.1 mm, vias 33 -> 34
- net FPDI_CEC: track 24.4 -> 22.8 mm
- net D2-: track 13.2 -> 14.2 mm
- net CONN27: track 10.0 -> 10.6 mm
Other:
- board size 65 x 34 mm -> 65.6 x 34 mm
