File: src/anice.kicad_pcb (KiCad board)
At the start: 4 copper layers, 65.6 x 34 mm, 118 parts, among them J1 Conn_02x20_Counter_Clockwise, J2 USB_C_Receptacle_USB2.0_14P, J3 USB_C_Receptacle_USB2.0_14P, J4 USB_C_Receptacle_USB2.0_14P, J5 HDMI_C_1.3, J6 Micro_SD_Card_Det1, U1 ECP5U_12_CABGA256, U10 W9825G6KH-6, U11 W25Q128JVS, U2 TLV62569DRL, U3 TLV62569DRL, U4 TLV62569DRL, U5 FT231XQ, U6 TPD2EUSB30, U7 TPD2EUSB30, U8 TPD2EUSB30, U9 PCA9306DC1, Y1 ECS-2520MV-xxx-xx

Commit message: Add annotations
Other:
- board text added: "Change files and layers on the right side!!! -> These two pcbs will be joined together physically Control+Scroll to zoom, Right click & drag to pan"
- board text removed: "Change files on the right side!!! -> These two pcbs will be joined together physically Scroll to zoom, Right click & drag to pan"
Changed lines of the file:
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@@
 		(layer "Edge.Cuts")
 	)
-	(gr_text "Change files on the right side!!! ->\nThese two pcbs will be joined together physically\n\nScroll to zoom,\nRight click & drag to pan"
+	(gr_text "Change files and layers on the right side!!! ->\nThese two pcbs will be joined together physically\n\nControl+Scroll to zoom,\nRight click & drag to pan"
 		(at 161.28 45.18 0)
 		(layer "Cmts.User")
@@
 			)
 		)
+	)
+	(zone
+		(net 0)
+		(net_name "")
+		(layers "F.Cu" "B.Cu" "In1.Cu" "In2.Cu")
+		(hatch edge 0.5)
+		(connect_pads
+			(clearance 0)
+		)
+		(min_thickness 0.25)
+		(filled_areas_thickness no)
+		(keepout
+			(tracks allowed)
+			(vias allowed)
+			(pads allowed)
+			(copperpour not_allowed)
+			(footprints allowed)
+		)
+		(placement
+			(enabled no)
+			(sheetname "/")
+		)
+		(fill
+			(thermal_gap 0.5)
+			(thermal_bridge_width 0.5)
+		)
+		(polygon
+			(pts
+				(xy 119.6 96.97) (xy 118.38 96.97) (xy 118.38 95.42) (xy 119.62 95.42)
+			)
+		)
