File: src/icedev.kicad_pcb (KiCad board)
At the start: 4 copper layers, 35.6 x 53.3 mm, 61 parts, among them J1 Conn_01x08, J10 Conn_01x18, J11 USB_C_Receptacle_PowerOnly_6P, J12 Conn_01x18, J2 Conn_02x01, J3 USB_C_Receptacle_USB2.0_14P, J4 Conn_02x01, J5 Conn_02x01, J7 Conn_02x02_Odd_Even, J8 Conn_01x03, J9 Conn_02x01, U1 ICE40UP5K-SG48ITR, U2 AMS1117-1.2, U3 AMS1117-3.3, U4 W25Q128JVS, U5 FM24C64B, U6 SRV05-4, X1 MPUOSC

Commit message: Structure project
Other:
- board text added: "Change files on the right side!!! -> These two pcbs will be joined together physically"
Changed lines of the file:
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@@
+		)
+	)
+	(gr_text "Change files on the right side!!! ->\nThese two pcbs will be joined together physically"
+		(at 159.65 29.17 0)
+		(layer "Cmts.User")
+		(effects
+			(font
+				(size 3 3)
+				(thickness 0.6)
+				(bold yes)
+			)
+			(justify left bottom)
 		)
 	)

Commit message: Tidy project
Other:
- board text added: "Change files on the right side!!! -> These two pcbs will be joined together physically Scroll to zoom, Right click & drag to pan"
- board text removed: "Change files on the right side!!! -> These two pcbs will be joined together physically"
Changed lines of the file:
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@@
 		)
 	)
-	(gr_text "Change files on the right side!!! ->\nThese two pcbs will be joined together physically"
-		(at 159.65 29.17 0)
+	(gr_text "Change files on the right side!!! ->\nThese two pcbs will be joined together physically\n\nScroll to zoom,\nRight click & drag to pan"
+		(at 161.01 44.9 0)
 		(layer "Cmts.User")
 		(effects

Commit message: Add annotations
Parts:
- removed G***: LOGO, LOGO
Other:
- board text added: "Change files and layers on the right side!!! -> These two pcbs will be joined together physically Control+Scroll to zoom, Right click & drag to pan"
- board text removed: "Change files on the right side!!! -> These two pcbs will be joined together physically Scroll to zoom, Right click & drag to pan"
