File: src/onlyanice/gdpi.kicad_sch (KiCad schematic)
At the start: 7 parts, among them J1 Conn_02x20_Counter_Clockwise, U1 ECP5U_12_CABGA256

Commit message: Structure project
Parts:
- removed C43: 100nF, Capacitor_SMD:C_0402_1005Metric, symbol Device:C
- removed H1, H2, H3, H4: MountingHole_Pad, MountingHole:MountingHole_2.5mm, symbol Mechanical:MountingHole
- removed J1: Conn_02x20_Counter_Clockwise, Connector_PinHeader_2.54mm:PinHeader_2x20_P2.54mm_Vertical, symbol Connector_Generic:Conn_02x20_Odd_Even
- removed U1: ECP5U_12_CABGA256, Package_BGA:BGA-256_14.0x14.0mm_Layout16x16_P0.8mm_Ball0.45mm_Pad0.32mm_NSMD, symbol josh-ic:ECP5U_12_CABGA256
- added C13, C14, C15, C16, C17, C18, C19, C20: 22nF, Capacitor_SMD:C_0603_1608Metric, symbol Device:C_Small
- added C21: 100pF, Capacitor_SMD:C_0603_1608Metric, symbol Device:C
- added C23, C39: 100nF, Capacitor_SMD:C_0402_1005Metric, symbol Device:C
- added C40: 15pF, Capacitor_SMD:C_0402_1005Metric, symbol Device:C
- added J7: HDMI_C_1.3, anice-lib:XKB Connection A71-05H4-111N1, symbol Connector:HDMI_C_1.3
- added R10, R8: 470, Resistor_SMD:R_0603_1608Metric, symbol Device:R
- added R11: 100k, Resistor_SMD:R_0603_1608Metric, symbol Device:R
- added R12, R13: 4.7k, Resistor_SMD:R_0603_1608Metric, symbol Device:R
- added R14, R15: 3.3k, Resistor_SMD:R_0603_1608Metric, symbol Device:R
- added R9: 10k, Resistor_SMD:R_0603_1608Metric, symbol Device:R
- added U1: ECP5U_12_CABGA256, Package_BGA:BGA-256_14.0x14.0mm_Layout16x16_P0.8mm_Ball0.45mm_Pad0.32mm_NSMD, symbol josh-ic:ECP5U_12_CABGA256
- added U9: PCA9306DC1, Package_SO:VSSOP-8_2.3x2mm_P0.5mm, symbol Interface:PCA9306DC1
- added Y1: ECS-2520MV-xxx-xx, Crystal:Crystal_SMD_3225-4Pin_3.2x2.5mm, symbol Oscillator:ECS-2520MV-xxx-xx
Connections:
- net +3V3: now also C23.2, C39.1, R14.1, R15.1, U1.K11 (VCCIO3[2]), U1.L11 (VCCIO3[2]), U9.2 (VREF1), U9.8 (EN), Y1.1 (Tri-State), Y1.4 (VDD)
- net +5V: now also J7.18 (+5V), R11.1, R12.1, R13.1
- net FPDI_SCL: now also R15.2, U9.3 (SCL1)
- net FPDI_SDA: now also R14.2, U9.4 (SDA1)
- net GND: now also C21.2, C23.1, C39.2, C40.2, J7.1 (D2S), J7.10 (CKS), J7.13 (GND), J7.4 (D1S), J7.7 (D0S), J7.SH, U9.1 (GND), Y1.2 (GND)
- new net: C21.1, R11.2, U9.7 (VREF2)
- new net: J7.19 (HPD), R10.1
- new net: C19.2, J7.11 (CK+)
- new net: C20.2, J7.12 (CK-)
- new net: J7.14 (CEC), R8.1
- new net: J7.17 (UTILITY), R9.1
- new net: C13.2, J7.2 (D2+)
- new net: C14.2, J7.3 (D2-)
- new net: C15.2, J7.5 (D1+)
- new net: C16.2, J7.6 (D1-)
- new net: C17.2, J7.8 (D0+)
- new net: C18.2, J7.9 (D0-)
- new net FPDI_CEC: R8.2, U1.T14 (PR41D/-/RDQ44)
- new net FPDI_CLK+: C19.1, U1.T15 (PR38D/-/RDQ44)
- new net FPDI_CLK-: C20.1, U1.R15 (PR38C/+/RDQ44)
- new net FPDI_D0+: C17.1, U1.P16 (PR35A/+/HS/RDQ32)
- new net FPDI_D0-: C18.1, U1.R16 (PR35B/-/VREF1_3/HS/RDQ32)
- new net FPDI_D1+: C15.1, U1.M16 (PR26C/+/PCLKT3_0/RDQ32)
- new net FPDI_D1-: C16.1, U1.M15 (PR26D/-/PCLKC3_0/RDQ32)
- new net FPDI_D2+: C13.1, U1.L16 (PR26A/+/PCLKT3_1/HS/RDQ32)
- new net FPDI_D2-: C14.1, U1.L15 (PR26B/-/PCLKC3_1/HS/RDQ32)
- new net FPDI_HPD: R10.2, U1.N16 (PR32A/+/HS/RDQS32)
- new net FPDI_UTIL: R9.2, U1.P15 (PR32B/-/HS/RDQSN32)
- new net GCLK: C40.1, U1.K13 (PR29A/+/GR_PCLK3_0/HS/RDQ32), Y1.3 (OUT)
- new net GPDI_SCL: J7.15 (SCL), R12.2, U9.6 (SCL2)
- new net GPDI_SDA: J7.16 (SDA), R13.2, U9.5 (SDA2)
Other:
- removed sheet Flash
- removed sheet GDPI
- removed sheet Power
- removed sheet SDRAM
- removed sheet USB
- company: Cyao -> (none)
- title: Anice -> (none)
